File: TaikoPcb.kicad_sch (KiCad schematic)
At the start: 0 parts

Commit message: Add schematic
Parts:
- added C1: C_Polarized, symbol Device:C_Polarized
- added J1, J2, J3: Screw_Terminal_01x04, TerminalBlock:TerminalBlock_Xinya_XY308-2.54-4P_1x04_P2.54mm_Horizontal, symbol Connector:Screw_Terminal_01x04
- added R1, R2, R3, R4, R5, R6, R7, R8: 100k, symbol Device:R
- added R9: 330, symbol Device:R
- added U1: ~, symbol esp32-s3-supermini:esp32-s3-supermini
- added U2, U3, U4, U5: DB107-G, DB107-G_CIP, symbol DB107-G_CIP:DB107-G
Connections:
- new net: R3.1, U3.3
- new net: R3.2, R4.1, U1.11 (GP9)
- new net: R7.1, U5.3
- new net: R7.2, R8.1, U1.13 (GP11)
- new net: J1.4 (Pin_4), U3.1
- new net: J1.3 (Pin_3), U3.2
- new net: J1.1 (Pin_1), U2.2
- new net: J1.2 (Pin_2), U2.1
- new net: R1.2, R2.1, U1.10 (GP8)
- new net: R5.2, R6.1, U1.12 (GP10)
- new net: J3.4 (Pin_4), U1.14 (GP12)
- new net: R9.1, U1.15 (GP13)
- new net: C1.1, J3.1 (Pin_1), U1.18 (5v)
- new net: J2.1 (Pin_1), U4.2
- new net: J2.2 (Pin_2), U4.1
- new net: J2.3 (Pin_3), U5.2
- new net: J2.4 (Pin_4), U5.1
- new net: R1.1, U2.3
- new net: R5.1, U4.3
- new net: J3.3 (Pin_3), R9.2
- new net GND: C1.2, J3.2 (Pin_2), R2.2, R4.2, R6.2, R8.2, U1.17 (GND), U2.4, U3.4, U4.4, U5.4
Other:
- note added: "Clk"
- note added: "Data"
- note added: "Gnd"
- note added: "V+"

Commit message: rewire
Connections:
- net at R3.2, R4.1: now also U1.6 (GP4); no longer U1.11 (GP9)
- net at R7.2, R8.1: now also U1.3 (GP1); no longer U1.13 (GP11)
- net at R1.2, R2.1: now also U1.7 (GP5); no longer U1.10 (GP8)
- net at R5.2, R6.1: now also U1.4 (GP2); no longer U1.12 (GP10)
- net at U1.14 (GP12): no longer J3.4 (Pin_4)
- net at U1.15 (GP13): no longer R9.1
- net at U1.8 (GP6): now also J3.4 (Pin_4)
- net at U1.9 (GP7): now also R9.1
Other:
- note added: "GP3 is not usable (strapping pin)"
- moved on the sheet: C1, J1, J2, J3, R1, R2, R3, R4, R5, R6, R7, R8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

Commit message: fill in most of PCB
Parts:
- C1: footprint (none) -> Diode_THT:D_DO-34_SOD68_P10.16mm_Horizontal
- R1, R2, R3, R4, R5, R6, R7, R8, R9: footprint (none) -> Resistor_THT:R_Axial_DIN0207_L6.3mm_D2.5mm_P7.62mm_Horizontal
- U1: value ~ -> ESP32-S3-Supermini; footprint (none) -> esp32-s3-supermini:esp32-s3-supermini
- U2, U3, U4, U5: footprint DB107-G_CIP -> DB107-G:DB107-G_CIP
Changed lines of the file:
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@@
 			)
 		)
-		(property "Footprint" ""
+		(property "Footprint" "Resistor_THT:R_Axial_DIN0207_L6.3mm_D2.5mm_P7.62mm_Horizontal"
 			(at 82.042 101.6 90)
 			(effects
@@
 			)
 		)
-		(property "Footprint" ""
+		(property "Footprint" "Resistor_THT:R_Axial_DIN0207_L6.3mm_D2.5mm_P7.62mm_Horizontal"
 			(at 141.732 101.6 90)
 			(effects
@@
 			)
 		)
-		(property "Footprint" "DB107-G_CIP"
+		(property "Footprint" "DB107-G:DB107-G_CIP"
 			(at 86.36 67.31 0)
 			(effects
@@
 		(fields_autoplaced yes)
 		(property "Reference" "U1"
-			(at 171.704 88.9 0)
-			(effects
-				(font
-					(size 1.27 1.27)
-				)
-			)
-		)
-		(property "Value" "~"
-			(at 171.704 91.44 0)
-			(effects
-				(font
-					(size 1.27 1.27)
-				)
-			)
-		)
-		(property "Footprint" ""
+			(at 171.704 92.964 0)
+			(effects
+				(font
+					(size 1.27 1.27)
+				)
+			)
+		)
+		(property "Value" "ESP32-S3-Supermini"
+			(at 171.704 95.504 0)
+			(effects
+				(font
+					(size 1.27 1.27)
+				)
+				(hide yes)
+			)
+		)
+		(property "Footprint" "esp32-s3-supermini:esp32-s3-supermini"
 			(at 181.61 116.84 0)
 			(effects
@@
 			)
 		)
-		(property "Footprint" "DB107-G_CIP"
+		(property "Footprint" "DB107-G:DB107-G_CIP"
 			(at 146.05 67.31 0)
 			(effects
@@
 			)
 		)
-		(property "Footprint" ""
+		(property "Footprint" "Resistor_THT:R_Axial_DIN0207_L6.3mm_D2.5mm_P7.62mm_Horizontal"
 			(at 112.522 124.46 90)
 			(effects
@@
 			)
 		)
-		(property "Footprint" ""
+		(property "Footprint" "Resistor_THT:R_Axial_DIN0207_L6.3mm_D2.5mm_P7.62mm_Horizontal"
 			(at 54.102 101.6 90)
 			(effects
@@
 			)
 		)
-		(property "Footprint" ""
+		(property "Footprint" "Resistor_THT:R_Axial_DIN0207_L6.3mm_D2.5mm_P7.62mm_Horizontal"
 			(at 82.042 124.46 90)
 			(effects
@@
 			)
 		)
-		(property "Footprint" "DB107-G_CIP"
+		(property "Footprint" "DB107-G:DB107-G_CIP"
 			(at 116.84 67.31 0)
 			(effects
@@
 			)
 		)
-		(property "Footprint" "DB107-G_CIP"
+		(property "Footprint" "DB107-G:DB107-G_CIP"
 			(at 58.42 67.31 0)
 			(effects
@@
 			)
 		)
-		(property "Footprint" ""
+		(property "Footprint" "Resistor_THT:R_Axial_DIN0207_L6.3mm_D2.5mm_P7.62mm_Horizontal"
 			(at 141.732 124.46 90)
 			(effects
@@
 			)
 		)
-		(property "Footprint" ""
+		(property "Footprint" "Diode_THT:D_DO-34_SOD68_P10.16mm_Horizontal"
 			(at 206.7052 105.41 0)
 			(effects
@@
 			)
 		)
-		(property "Footprint" ""
+		(property "Footprint" "Resistor_THT:R_Axial_DIN0207_L6.3mm_D2.5mm_P7.62mm_Horizontal"
 			(at 215.138 113.03 90)
 			(effects
@@
 			)
 		)
-		(property "Footprint" ""
+		(property "Footprint" "Resistor_THT:R_Axial_DIN0207_L6.3mm_D2.5mm_P7.62mm_Horizontal"
 			(at 112.522 101.6 90)
 			(effects
@@
 			)
 		)
-		(property "Footprint" ""
+		(property "Footprint" "Resistor_THT:R_Axial_DIN0207_L6.3mm_D2.5mm_P7.62mm_Horizontal"
 			(at 54.102 124.46 90)
 			(effects
