File: TaikoPcb.kicad_pcb (KiCad board)
At the start: 2 copper layers, 65.5 x 51.5 mm, 21 parts, among them J1 Screw_Terminal_01x04, J2 Screw_Terminal_01x04, J3 Screw_Terminal_01x04, U1 ESP32-S3-Supermini, U2 DB107-G, U3 DB107-G, U4 DB107-G, U5 DB107-G

Commit message: New gerbers, remove jlcjlcjlcjlc
Other:
- board text added: "v1.0"
- board text removed: "JLCJLCJLCJLC"
Changed lines of the file:
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@@
 		)
 	)
-	(gr_text "JLCJLCJLCJLC"
-		(at 172.5 44.5 270)
+	(gr_text "ESP32\nS3\nSuperMini"
+		(at 166 72.5 0)
 		(layer "B.SilkS")
 		(effects
@@
 				(bold yes)
 			)
-			(justify left bottom mirror)
+			(justify bottom mirror)
 		)
 	)
-	(gr_text "ESP32\nS3\nSuperMini"
-		(at 166 72.5 0)
+	(gr_text "v1.0"
+		(at 166.2 76.5 0)
 		(layer "B.SilkS")
 		(effects
